File: MCU Datalogger.kicad_sch (KiCad schematic)
At the start: 25 parts, among them U1 24LC1025, U2 24LC1025, U3 DS1337S_, U4 ATMEGA328P-AU, Y1 32.768 KHz, Y2 16 MHz

Commit message: Setup Pcbnew.
Changed lines of the file:
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@@
 			(font
 				(size 1.27 1.27)
-				(thickness 0.254)
-				(bold yes)
+				(thickness 0.1588)
 			)
 			(justify left top)
@@
 			(font
 				(size 1.27 1.27)
-				(thickness 0.254)
-				(bold yes)
+				(thickness 0.1588)
 			)
 			(justify left top)
@@
 			(font
 				(size 1.27 1.27)
-				(thickness 0.254)
-				(bold yes)
+				(thickness 0.1588)
 			)
 			(justify left top)
@@
 	(wire
 		(pts
-			(xy 200.66 129.54) (xy 209.55 129.54)
+			(xy 203.2 129.54) (xy 212.09 129.54)
 		)
 		(stroke
@@
 	(wire
 		(pts
-			(xy 200.66 125.73) (xy 205.74 125.73)
+			(xy 203.2 125.73) (xy 208.28 125.73)
 		)
 		(stroke
@@
 	)
 	(label "D2"
-		(at 177.8 129.54 180)
+		(at 180.34 129.54 180)
 		(effects
 			(font
@@
 	)
 	(label "RX"
-		(at 200.66 143.51 0)
+		(at 203.2 143.51 0)
 		(effects
 			(font
@@
 	)
 	(label "D3"
-		(at 177.8 133.35 180)
+		(at 180.34 133.35 180)
 		(effects
 			(font
@@
 	)
 	(label "RESET"
-		(at 200.66 156.21 0)
+		(at 203.2 156.21 0)
 		(effects
 			(font
@@
 	)
 	(label "TX"
-		(at 200.66 140.97 0)
+		(at 203.2 140.97 0)
 		(effects
 			(font
@@
 	)
 	(label "SDA"
-		(at 200.66 133.35 0)
+		(at 203.2 133.35 0)
 		(effects
 			(font
@@
 	)
 	(label "D5"
-		(at 177.8 140.97 180)
+		(at 180.34 140.97 180)
 		(effects
 			(font
@@
 	)
 	(label "D8"
-		(at 177.8 152.4 180)
+		(at 180.34 152.4 180)
 		(effects
 			(font
@@
 	)
 	(label "SCK"
-		(at 200.66 135.89 0)
+		(at 203.2 135.89 0)
 		(effects
 			(font
@@
 	)
 	(label "D4"
-		(at 177.8 137.16 180)
+		(at 180.34 137.16 180)
 		(effects
 			(font
@@
 	)
 	(label "MOSI"
-		(at 200.66 151.13 0)
+		(at 203.2 151.13 0)
 		(effects
 			(font
@@
 	)
 	(label "Vcc"
-		(at 205.74 125.73 0)
+		(at 208.28 125.73 0)
 		(effects
 			(font
@@
 	)
 	(label "D7"
-		(at 177.8 148.59 180)
+		(at 180.34 148.59 180)
 		(effects
 			(font
@@
 	)
 	(label "D6"
-		(at 177.8 144.78 180)
+		(at 180.34 144.78 180)
 		(effects
 			(font
@@
 	)
 	(label "MISO"
-		(at 200.66 148.59 0)
+		(at 203.2 148.59 0)
 		(effects
 			(font
@@
 	(symbol
 		(lib_id "power:GND")
-		(at 209.55 129.54 0)
+		(at 212.09 129.54 0)
 		(unit 1)
 		(exclude_from_sim no)
@@
 		(fields_autoplaced yes)
 		(property "Reference" "#PWR010"
-			(at 209.55 135.89 0)
+			(at 212.09 135.89 0)
 			(effects
 				(font
@@
 		)
 		(property "Value" "GND"
-			(at 209.55 134.62 0)
+			(at 212.09 134.62 0)
 			(effects
 				(font
@@
 		)
 		(property "Footprint" ""
-			(at 209.55 129.54 0)
+			(at 212.09 129.54 0)
 			(effects
 				(font
@@
 		)
 		(property "Datasheet" ""
-			(at 209.55 129.54 0)
+			(at 212.09 129.54 0)
 			(effects
 				(font
@@
 		)
 		(property "Description" "Power symbol creates a global label with name \"GND\" , ground"
-			(at 209.55 129.54 0)
+			(at 212.09 129.54 0)
 			(effects
 				(font
@@
 	)
 	(sheet
-		(at 177.8 123.825)
+		(at 180.34 123.825)
 		(size 22.86 34.925)
 		(exclude_from_sim no)
@@
 		)
 		(property "Sheetname" "connectors"
-			(at 177.8 123.1134 0)
+			(at 180.34 123.1134 0)
 			(effects
 				(font
@@
 		)
 		(property "Sheetfile" "connectors.kicad_sch"
-			(at 177.8 159.3346 0)
+			(at 180.34 159.3346 0)
 			(effects
 				(font
@@
 		)
 		(pin "SDA" bidirectional
-			(at 200.66 133.35 0)
+			(at 203.2 133.35 0)
 			(effects
 				(font
@@
 		)
 		(pin "TX" output
-			(at 200.66 140.97 0)
+			(at 203.2 140.97 0)
 			(effects
 				(font
@@
 		)
 		(pin "RX" input
-			(at 200.66 143.51 0)
+			(at 203.2 143.51 0)
 			(effects
 				(font
@@
 		)
 		(pin "D4" bidirectional
-			(at 177.8 137.16 180)
+			(at 180.34 137.16 180)
 			(effects
 				(font
@@
 		)
 		(pin "D2" bidirectional
-			(at 177.8 129.54 180)
+			(at 180.34 129.54 180)
 			(effects
 				(font
@@
 		)
 		(pin "D3" bidirectional
-			(at 177.8 133.35 180)
+			(at 180.34 133.35 180)
 			(effects
 				(font
@@
 		)
 		(pin "D5" bidirectional
-			(at 177.8 140.97 180)
+			(at 180.34 140.97 180)
 			(effects
 				(font
@@
 		)
 		(pin "D6" bidirectional
-			(at 177.8 144.78 180)
+			(at 180.34 144.78 180)
 			(effects
 				(font
@@
 		)
 		(pin "D7" bidirectional
-			(at 177.8 148.59 180)
+			(at 180.34 148.59 180)
 			(effects
 				(font
@@
 		)
 		(pin "D8" bidirectional
-			(at 177.8 152.4 180)
+			(at 180.34 152.4 180)
 			(effects
 				(font
@@
 		)
 		(pin "MISO" output
-			(at 200.66 148.59 0)
+			(at 203.2 148.59 0)
 			(effects
 				(font
@@
 		)
 		(pin "SCK" passive
-			(at 200.66 135.89 0)
+			(at 203.2 135.89 0)
 			(effects
 				(font
@@
 		)
 		(pin "Vcc" passive
-			(at 200.66 125.73 0)
+			(at 203.2 125.73 0)
 			(effects
 				(font
@@
 		)
 		(pin "GND" passive
-			(at 200.66 129.54 0)
+			(at 203.2 129.54 0)
 			(effects
 				(font
@@
 		)
 		(pin "MOSI" input
-			(at 200.66 151.13 0)
+			(at 203.2 151.13 0)
 			(effects
 				(font
@@
 		)
 		(pin "RESET" passive
-			(at 200.66 156.21 0)
+			(at 203.2 156.21 0)
 			(effects
 				(font

Commit message: Fixed outstanding issues.
Connections:
- net Vcc: now also BT1.1 (+), C5.1, D1.2 (A), U4.18 (AVCC)
Changed lines of the file:
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@@
+		)
+	)
+	(label "Vcc"
+		(at 256.54 45.72 0)
+		(effects
+			(font
+				(size 1.27 1.27)
+			)
+			(justify left bottom)
 		)
 	)

Commit message: Fixed two defects in the schematic.
Connections:
- net SCK: no longer R3.2, U1.6 (SCL), U2.6 (SCL), U3.6 (SCL), U4.28 (PC5)
- new net SCL: R3.2, U1.6 (SCL), U2.6 (SCL), U3.6 (SCL), U4.28 (PC5)
Other:
- sheet connectors ports: added SCL; removed none
Changed lines of the file:
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@@
 	(wire
 		(pts
-			(xy 240.03 40.64) (xy 240.03 45.72)
-		)
-		(stroke
-			(width 0)
-			(type default)
-		)
-	)
-	(wire
-		(pts
 			(xy 99.06 144.78) (xy 99.06 148.59)
 		)
@@
 		)
 	)
+	(label "SCK"
+		(at 203.2 139.7 0)
+		(effects
+			(font
+				(size 1.27 1.27)
+			)
+			(justify left bottom)
+		)
+	)
 	(label "SDA"
 		(at 43.18 63.5 180)
@@
 	)
 	(label "RX"
-		(at 203.2 143.51 0)
+		(at 203.2 144.78 0)
 		(effects
 			(font
@@
 	)
 	(label "TX"
-		(at 203.2 140.97 0)
+		(at 203.2 142.24 0)
 		(effects
 			(font
@@
 		)
 	)
-	(label "SCK"
+	(label "SCL"
 		(at 182.88 88.9 180)
 		(effects
@@
 		)
 	)
-	(label "SCK"
+	(label "SCL"
 		(at 49.53 143.51 0)
 		(effects
@@
 		)
 	)
-	(label "SCK"
+	(label "SCL"
 		(at 203.2 135.89 0)
 		(effects
@@
 		)
 	)
-	(label "SCK"
+	(label "SCL"
 		(at 43.18 55.88 180)
 		(effects
@@
 		)
 	)
-	(label "SCK"
+	(label "SCL"
 		(at 85.09 143.51 0)
 		(effects
@@
 		)
 	)
-	(label "SCK"
+	(label "SCL"
 		(at 99.06 148.59 0)
 		(effects
@@
 	)
 	(symbol
-		(lib_id "power:PWR_FLAG")
-		(at 240.03 40.64 0)
-		(unit 1)
-		(exclude_from_sim no)
-		(in_bom yes)
-		(on_board yes)
-		(dnp no)
-		(fields_autoplaced yes)
-		(property "Reference" "#FLG01"
-			(at 240.03 38.735 0)
-			(effects
-				(font
-					(size 1.27 1.27)
-				)
-				(hide yes)
-			)
-		)
-		(property "Value" "PWR_FLAG"
-			(at 240.03 35.56 0)
-			(effects
-				(font
-					(size 1.27 1.27)
-				)
-			)
-		)
-		(property "Footprint" ""
-			(at 240.03 40.64 0)
-			(effects
-				(font
-					(size 1.27 1.27)
-				)
-				(hide yes)
-			)
-		)
-		(property "Datasheet" "~"
-			(at 240.03 40.64 0)
-			(effects
-				(font
-					(size 1.27 1.27)
-				)
-				(hide yes)
-			)
-		)
-		(property "Description" "Special symbol for telling ERC where power comes from"
-			(at 240.03 40.64 0)
-			(effects
-				(font
-					(size 1.27 1.27)
-				)
-				(hide yes)
-			)
-		)
-		(pin "1"
-		)
-		(instances
-			(project ""
-				(path "/95e137fe-1751-439b-90d7-a721ce4736b3"
-					(reference "#FLG01")
-					(unit 1)
-				)
-			)
-		)
-	)
-	(symbol
 		(lib_id "power:GND")
 		(at 81.28 76.2 0)
@@
 		)
 		(pin "TX" output
-			(at 203.2 140.97 0)
+			(at 203.2 142.24 0)
 			(effects
 				(font
@@
 		)
 		(pin "RX" input
-			(at 203.2 143.51 0)
+			(at 203.2 144.78 0)
 			(effects
 				(font
@@
 			)
 		)
-		(pin "SCK" passive
-			(at 203.2 135.89 0)
-			(effects
-				(font
-					(size 1.27 1.27)
-				)
-				(justify right)
-			)
-		)
 		(pin "Vcc" passive
 			(at 203.2 125.73 0)
@@
 			(effects
 				(font
+					(size 1.27 1.27)
+				)
+				(justify right)
+			)
+		)
+		(pin "SCL" passive
+			(at 203.2 135.89 0)
+			(effects
+				(font
+					(size 1.27 1.27)
+				)
+				(justify right)
+			)
+		)
+		(pin "SCK" passive
+			(at 203.2 139.7 0)
+			(effects
+				(font
